File: DashcamPower.kicad_sch (KiCad schematic)
At the start: 22 parts, among them J1 USB_C_Receptacle_USB2.0_16P, J2 USB_C_Receptacle_USB2.0_16P, Q1 IRLML6402, Q2 MMBT5551L, U1 XC6206P332MR-G, U2 LSM6DS3, U3 RP2040, U4 W25Q128JVS

Commit message: Sync to server
Changes on desktop
Parts:
- added C10, C13, C7, C8: 100n, Capacitor_SMD:C_0603_1608Metric, symbol Device:C
- added C11, C12: 15p, Capacitor_SMD:C_0603_1608Metric, symbol Device:C
- added C6, C9: 1u 50V, Capacitor_SMD:C_0805_2012Metric, symbol Device:C
- added D1: Green 0805, LED_SMD:LED_0805_2012Metric, symbol Device:LED
- added D2: Red 0805, LED_SMD:LED_0805_2012Metric, symbol Device:LED
- added D3: Yellow 0805, LED_SMD:LED_0805_2012Metric, symbol Device:LED
- added J4: Conn_01x06, Connector_PinHeader_2.54mm:PinHeader_1x06_P2.54mm_Vertical, symbol Connector_Generic:Conn_01x06
- added LS1: Speaker_Crystal, symbol Device:Speaker_Crystal
- added R10: 1k, Resistor_SMD:R_0603_1608Metric, symbol Device:R
- added R11, R12, R17: 5.1k, Resistor_SMD:R_0603_1608Metric, symbol Device:R
- added R13: NF, Resistor_SMD:R_0603_1608Metric, symbol Device:R
- added R14, R15, R16, R18: 270R, Resistor_SMD:R_0603_1608Metric, symbol Device:R
- added SW1: B3FS-1000P, Button_Switch_SMD:SW_SPST_Omron_B3FS-100xP, symbol Switch:SW_Omron_B3FS
- added Y1: X322512MSB4SI, Crystal:Crystal_SMD_Abracon_ABM8AIG-4Pin_3.2x2.5mm, symbol Device:Crystal_GND24
- C1: Part CL21A475KAQNNNE -> C1779
- C2: Part CL21B105KBFNNNE -> C28323
- C4, C5: value 100nF -> 100n; Part CL05B104KO5NNNC -> C14663
- U1: Part XC6206P332MR-G# -> C5446
- U2: Part LSM6DS3TR -> C95230
- U4: Part W25Q128JVSIQ -> C97521
Connections:
- net +3.3V: now also U3.1 (IOVDD), U3.10 (IOVDD), U3.22 (IOVDD), U3.33 (IOVDD), U3.42 (IOVDD), U3.43 (ADC_AVDD), U3.44 (VREG_IN), U3.48 (USB_VDD), U3.49 (IOVDD), U4.8 (VCC), C10.1, C7.1, C8.1, C9.1, J4.6 (Pin_6), R17.1
- net GND: now also U3.57 (GND), U4.4 (GND), C10.2, C11.2, C12.2, C13.2, C6.2, C7.2, C8.2, C9.2, J4.2 (Pin_2), R14.2, R15.2, R16.2, SW1.2, Y1.2, Y1.4
- net I2C_SCL: now also U3.5 (GPIO3)
- net I2C_SDA: now also U3.4 (GPIO2)
- net IMU_INT1: now also U3.7 (GPIO5)
- net IMU_INT2: now also U3.8 (GPIO6)
- net QSPI_CLK: now also U4.6 (CLK)
- net QSPI_SD0: now also U4.5 (DI/IO_{0})
- net QSPI_SD1: now also U4.2 (DO/IO_{1})
- net QSPI_SD2: now also U4.3 (~{WP}/IO_{2})
- net QSPI_SD3: now also U4.7 (~{HOLD}/~{RESET}/IO_{3})
- net QSPI_SS: now also U4.1 (~{CS})
- net USB_OUT_ON: now also U3.2 (GPIO0)
- net BTN: now reaches U3.11 (GPIO8)
- net BTN: now also C13.1, R18.2
- net at U3.20 (XIN): now also C12.1, Y1.3
- net at U3.21 (XOUT): now also R10.2
- net at U3.23 (DVDD), U3.50 (DVDD): now also U3.45 (VREG_VOUT), C6.1
- net SWC: now reaches U3.24 (SWCLK)
- net SWC: now also J4.3 (Pin_3)
- net SWD: now reaches U3.25 (SWD)
- net SWD: now also J4.1 (Pin_1)
- net LED_G: now reaches U3.32 (GPIO21)
- net LED_G: now also D1.2 (A)
- net LED_R: now reaches U3.35 (GPIO23)
- net LED_R: now also D2.2 (A)
- net LED_Y: now reaches U3.37 (GPIO25)
- net LED_Y: now also D3.2 (A)
- net at C3.1, J2.A4 (VBUS), J2.A9 (VBUS)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: now also R11.1, R12.1
- net at J2.A5 (CC1): now also R12.2
- net at J2.A6 (D+): now also J2.B6 (D+), R13.2
- net at J2.A7 (D-): now also J2.B7 (D-), R13.1
- net at J2.B5 (CC2): now also R11.2
- new net: R17.2, R18.1, SW1.1
- new net: C11.1, R10.1, Y1.1
- new net: D3.1 (K), R16.1
- new net: D2.1 (K), R15.1
- new net: D1.1 (K), R14.1
- new net URX: J4.5 (Pin_5)
- new net UTX: J4.4 (Pin_4)
Other:
- note added: "Check footprint is correct"
- note added: "To add:"
- note added: "beeper"
- note added: "button(s)"
- moved on the sheet: C1, C2, C3, J1, J2, Q1, Q2, R1, R2, R3, R4, R5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

Commit message: PCB draft
Parts:
- added C14, C15: 100n, Capacitor_SMD:C_0603_1608Metric, symbol Device:C
- added Q3: MMBT5551L, Package_TO_SOT_SMD:SOT-23, symbol Transistor_BJT:MMBT5551L
- added R19, R21: 5.1k, Resistor_SMD:R_0603_1608Metric, symbol Device:R
- added R20: 0R, Resistor_SMD:R_0805_2012Metric, symbol Device:R
- added R22: 270R, Resistor_SMD:R_0603_1608Metric, symbol Device:R
- LS1: footprint (none) -> Connector_Wire:SolderWire-0.1sqmm_1x02_P3.6mm_D0.4mm_OD1mm
Connections:
- net +3.3V: now also R21.1
- net +5V: now also R20.1
- net GND: now also C14.2, Q3.2 (E)
- net BUZZER: now reaches U3.17 (GPIO14)
- net BUZZER: now also R19.1
- net at U3.26 (RUN): now also C14.1, R21.2
- net USB_RES_D_P: now reaches R9.1, U3.46 (USB_DM)
- net USB_RES_D_N: now reaches R8.2, U3.47 (USB_DP)
- net at LS1.1: now also R20.2
- net at LS1.2: now also Q3.3 (C)
- net at C3.1, J2.A4 (VBUS), J2.A9 (VBUS)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: now also C15.1
- net at Q1.1 (G), R3.2: now also C15.2, R22.2; no longer Q2.3 (C)
- new net: Q3.1 (B), R19.2
- new net: Q2.3 (C), R22.1
- no-connect marks 0 -> 21
Other:
- note removed: "beeper"
- moved on the sheet: LS1, Q1, Q2, R3, R4, R8, R9
